File: hardware/basic/top/Tek-BASIC-TOP.sch (EAGLE design)
At the start: 0 parts

Commit message: Upload ot the udpdates made on the top board design: base items added on the schematic and on the board
Parts:
- added C10, C11: 300p, LinnesLab-Passives:CAPACITOR0603
- added C12: 10u, LinnesLab-Passives:CAPACITOR0805
- added C13, C15: 4.7u, LinnesLab-Passives:CAPACITOR0603
- added C14: 100n, LinnesLab-Passives:CAPACITOR0603
- added C17, C5, C6, C7: 1u, LinnesLab-Passives:CAPACITOR0603
- added C21, C22, C24, C25, C26: 2.2uF, LinnesLab-Passives:CAPACITOR0402
- added C23: 10uF, LinnesLab-Passives:CAPACITOR0603
- added C8, C9: (no value), LinnesLab-Passives:CAPACITOR0603
- added CHRG2: MCP73831, LinnesLab-Power:MCP73831
- added CORTEX1: CORTEX_DEBUG_PTH, LinnesLab-Connectors:CORTEX_DEBUG_PTH
- added D1, D4, D5: (no value), LinnesLab-DiscreteSemi:SCHOTTKY-USC
- added J2: (no value), LinnesLab-Connectors:CONN_02
- added L2: 10u, LinnesLab-Passives:INDUCTOR0603
- added LDO2: MIC5504, LinnesLab-Power:MIC5504
- added LED3: RED, LinnesLab-LED:LED0603
- added LED4: BLUE, LinnesLab-LED:LED0603
- added R10: 390k, LinnesLab-Passives:RESISTOR0603
- added R11: (no value), LinnesLab-Passives:RESISTOR0603
- added R12, R13, R14, R15: 100k, LinnesLab-Passives:RESISTOR0603
- added R18, R19, R5, R9: 10k, LinnesLab-Passives:RESISTOR0603
- added R3, R4: 1k, LinnesLab-Passives:RESISTOR0603
- added SD2: (no value), LinnesLab-Connectors:MICROSD
- added SW1, SW2, SW5: SWITCH.MOM, LinnesLab-Switches:SWITCH.MOM
- added SW3, SW4: (no value), LinnesLab-Switches:SPST-PTS830GG140-COPY.1-3
- added U2: NRF52832_MODULE_MDBT42, LinnesLab-Microcontrollers:NRF52832_MODULE_MDBT42
- added U3: PCF8523, LinnesLab-Clocks:PCF8523
- added U4: (no value), LinnesLab-Displays:DISP_OLED_UG-2864HSWEG01-NO-WRAPAROUND
- added USB2: USB.MICRO-BIGGERPADS, LinnesLab-Connectors:USB.MICRO-BIGGERPADS
- added XTAL2: 32.768kHz, LinnesLab-Clocks:CRYSTALECS-.327-12.5-12-C-TR
- added XTAL3: 32.7680kHz, LinnesLab-Clocks:CRYSTALECS-.327-12.5-12-C-TR
Connections:
- new net 3.3V: C12.2, C17.1, C24.2, C26.2, C6.1, CORTEX1.VCC, D1.C, LDO2.OUT, R15.2, R18.2, R19.2, R5.2, SD2.VDD, U2.VDD, U3.VDD, U4.VBAT, U4.VDD
- new net BATT: R13.1, R14.2
- new net CD1: SD2.CARD_DETECT
- new net CD2: SD2.CARD_DETECT1
- new net CHRG.STAT: CHRG2.STAT, R12.1
- new net CS.OLED: U4./CS
- new net DC.OLED: U4.DC/I2C_SA0
- new net DFU: SW3.B, U2.P0.20
- new net DTR: C14.1
- new net FRST: U2.P0.22
- new net GND: C10.2, C11.2, C12.1, C13.2, C15.1, C17.2, C23.1, C24.1, C25.1, C26.1, C5.1, C6.2, C7.2, C8.1, C9.2, CHRG2.VSS, CORTEX1.GND@3, CORTEX1.GND@5, CORTEX1.GNDDTCT, CORTEX1.KEY, J2.1, LDO2.GND, LED3.C, LED4.C, R10.2, R11.1, R14.1, R15.1, R9.1, SD2.GND, SD2.GND1, SD2.VSS, SW3.A, SW4.B, U2.GND@1, U2.GND@2, U2.GND@3, U2.GND@4, U3.VSS, U4.BS0, U4.BS2, U4.NC(GND)@1, U4.NC(GND)@2, U4.VLSS, U4.VSS, USB2.GND
- new net LED1: R3.2, U2.P0.17
- new net LED2: R4.2, U2.P0.19
- new net MISO: SD2.DATA_OUT, U2.P0.14
- new net MOSI: SD2.DATA_IN, U2.P0.13, U4.D1/SPI_SDIN/I2C_SDA
- new net N$1: CHRG2.PROG, R11.2
- new net N$10: LED4.A, R4.1
- new net N$11: L2.1, U2.DCC
- new net N$12: C7.1, L2.2, U2.DEC4
- new net N$14: CORTEX1.NC/TDI
- new net N$15: R9.2, U4.BS1
- new net N$16: R10.1, U4.IREF
- new net N$17: C21.2, U4.C2P
- new net N$18: C21.1, U4.C2N
- new net N$19: C22.2, U4.C1P
- new net N$20: C22.1, U4.C1N
- new net N$21: C23.2, U4.VCC
- new net N$23: C25.2, U4.VCOMH
- new net N$4: C8.2, U2.P0.00/XL1, XTAL2.1
- new net N$5: U3.OSCO, XTAL3.1
- new net N$6: C9.1, U2.P0.01/XL2, XTAL2.2
- new net N$7: U3.OSCI, XTAL3.2
- new net N$9: LED3.A, R3.1
- new net P0.09/NFC1: C11.1, U2.P0.09
- new net P0.10/NFC2: C10.1, U2.P0.10
- new net RESET: C14.2, CORTEX1.!RESET, D1.A, R5.1, SW4.A, U2.P0.21/RESET
- new net RESET.OLED: U4./RES
- new net RXD: U2.P0.08
- new net SCK: SD2.SCLK, U2.P0.12, U4.D0/SPI_SCLK/I2C_SCK
- new net SCL: R18.1, U2.P0.26, U3.SCL
- new net SD.CS: SD2.CS
- new net SDA: R19.1, U2.P0.25, U3.SDA
- new net SWCLK: CORTEX1.SWDCLK/TCK, U2.SWDCLK
- new net SWDIO: CORTEX1.SWDIO/TMS, U2.SWDIO
- new net SWO: CORTEX1.SWO/TDO, U2.P0.18/SWO
- new net TXD: U2.P0.06
- new net USB+: USB2.D+
- new net USB-: USB2.D-
- new net VBATT: U3.VBAT
- new net VIN: C15.2, C5.2, CHRG2.VIN, D4.C, D5.C, LDO2.EN, LDO2.IN, R12.2
- new net VLIPO: C13.1, CHRG2.VBAT, D4.A, J2.2, R13.2
- new net V_USB: D5.A, USB2.V+
Other:
- note added: "100nF+10K @ 3.3V = ~1.2ms to 0.7VCC"
- note added: "Additional notes for advanced users only"
- note added: "Back-up battery if desired"
- note added: "Connect MISO, MOSI, and SCK to appropriate pins on microcontroller. Those are SPI pins and are generally prespecified. You have more flexibility with the SD.CS pin."
- note added: "I2C Address = 0x68h"
- note added: "Microcontroller Reset Circuit"
- note added: "OLED"
- note added: "PIN_DFU / P0.20: If this pin is detected to be at GND level at startup, the board will enter a special serial bootloader mode and will not execute any user code, going straight into bootloader mode. If you wish to use this pin as a standard GPIO, make sure that it is pulled high with a pullup resistor so that your code will execute normally when the MCU starts up. FRST/P0.22: Setting this pin to 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"
- note added: "SPECIAL / PORT / PIN ON PACKAGE / GPIO(D_or_A) / Comments Factory Reset / P0.22 / pin38 / DO NOT USE FOR ANY GPIO SWDIO / none / pin37 / reserved-not available for general GPIO SWCLK / none / pin36 / reserved-not available for general GPIO RESET / P0.21 / pin35 / reserved-not available for general GPIO DFU / P0.20 / pin34 / reserved-not available for general GPIO LED2 / P0.19 / pin33 / reserved f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"
- note added: "SPECIAL / PORT / PIN ON PACKAGE / GPIO(D_or_A) / Comments SDA / P0.25 / pin2 / D25 SCL / P0.26 / pin3 / D26 none / P0.27 / pin4 / D27 none / P0.28 / pin5 / D28_or_A4 / (low drive, low frequency IO) none / P0.29 / pin6 / D29_or_A5 / (low drive, low frequency IO) none / P0.30 / pin7 / D30_or_A6 none / P0.31 / pin8 / D31_or_A7 / (used for battery level monitoring on Adafruit boards)"
- note added: "SPECIAL / PORT / PIN ON PACKAGE / GPIO(D_or_A) / Comments none / P0.02 / pin15 / D2_or_A0 none / P0.03 / pin16 / D3_or_A1 none / P0.04 / pin17 / D4_or_A2 none / P0.05 / pin18 / D5_or_A3 TXD / P0.06 / pin19 / D6 / but reserved for Serial communication and programming none / P0.07 / pin20 / D7 RXD / P0.08 / pin21 / D8 / but reserved for Serial communication and programming NFC1 / P0.09 / pin22 / D9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"
- note added: "Some pins are noted as reserved and not available for general GPIO (unless you are an adavanced user) I2C, SPI, and SWD pins can be repurposed if you know what you are doing For Milestones, avoid repurposing NFC pins. For P0.19 (LED2), Adafruit's Bluetooth Low Energy libraries use this pin to indicated successful pairing. The LED blinks when the device is doing some Bluetooth process and stays li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"
